File: kicad/PARTYLand_miniplayfield.kicad_pcb (KiCad board)
At the start: 2 copper layers, 71 parts, among them P1 CONN_6, U1 74HC595, U2 74HC595, U3 74HC595, U4 74HC595

Commit message: Finished placing all LEDs in the miniplayfield schematics and pcb layout. Also added propper PCB cut edges and ground planes for copper fill.
Parts:
- removed the G*** at (125.0, 204.2)
- added D33: 3RD, LEDs:LED-3MM, F.Cu at (98.8, 191.4)
- added D34: 2ND, LEDs:LED-3MM, F.Cu at (93.5, 174.8)
- added D35: 1ST, LEDs:LED-3MM, F.Cu at (88.9, 159.4)
- added D36: LEFT_CLOWN_EYE, LEDs:LED-3MM, F.Cu at (99.5, 171.2)
- added D37: RIGHT_CLOWN_EYE, LEDs:LED-3MM, F.Cu at (111.3, 167.4)
- added D38: MAD_D, LEDs:LED-3MM, F.Cu at (70.1, 158.1)
- added D39: MAD_A, LEDs:LED-3MM, F.Cu at (66.4, 139.5)
- added D40: MAD_M, LEDs:LED-3MM, F.Cu at (67.2, 120.3)
- added D41: DROP_ZONE, LEDs:LED-3MM, F.Cu at (59.6, 91.9)
- added D42: ARCADE, LEDs:LED-3MM, F.Cu at (111.8, 132.1)
- added D43: 5X, LEDs:LED-3MM, F.Cu at (123.4, 168.1)
- added D44: DRAGON_EYES, LEDs:LED-3MM, F.Cu at (173.6, 197.2)
- added D45: PUKE_P, LEDs:LED-3MM, F.Cu at (116.5, 90.0)
- added D46: PUKE_U, LEDs:LED-3MM, F.Cu at (129.3, 91.2)
- added D47: PUKE_K, LEDs:LED-3MM, F.Cu at (141.3, 91.2)
- added D48: PUKE_E, LEDs:LED-3MM, F.Cu at (154.7, 89.9)
- added D49: 1M, LEDs:LED-3MM, F.Cu at (127.6, 177.1)
- added D50: 3M, LEDs:LED-3MM, F.Cu at (148.5, 170.6)
- added D51: 5M, LEDs:LED-3MM, F.Cu at (161.7, 157.8)
- added D52: JACKPOT, LEDs:LED-3MM, F.Cu at (146.9, 249.5)
- added D53: EXTRABALL, LEDs:LED-3MM, F.Cu at (153.9, 237.3)
- added D54: DRAGON_5M, LEDs:LED-3MM, F.Cu at (160.9, 225.2)
- added D55: BONUS_X6, LEDs:LED-3MM, F.Cu at (151.6, 288.8)
- added D56: BONUS_X8, LEDs:LED-3MM, F.Cu at (162.5, 281.9)
- added R33: R, Discret:R3, F.Cu at (87.6, 170.2)
- added R34: R, Discret:R3, F.Cu at (83.8, 170.2)
- added R35: R, Discret:R3, F.Cu at (80.0, 170.2)
- added R36: R, Discret:R3, F.Cu at (76.2, 170.2)
- added R37: R, Discret:R3, F.Cu at (72.4, 170.2)
- added R38: R, Discret:R3, F.Cu at (68.6, 170.2)
- added R39: R, Discret:R3, F.Cu at (61.0, 170.2)
- added R40: R, Discret:R3, F.Cu at (57.1, 170.2)
- added R41: R, Discret:R3, F.Cu at (113.0, 108.0)
- added R42: R, Discret:R3, F.Cu at (119.4, 110.5)
- added R43: R, Discret:R3, F.Cu at (125.7, 113.0)
- added R44: R, Discret:R3, F.Cu at (132.1, 115.6)
- added R45: R, Discret:R3, F.Cu at (139.7, 115.6)
- added R46: R, Discret:R3, F.Cu at (146.1, 113.0)
- added R47: R, Discret:R3, F.Cu at (152.4, 110.5)
- added R48: R, Discret:R3, F.Cu at (158.8, 108.0)
- added R49: R, Discret:R3, F.Cu at (134.6, 165.1)
- added R50: R, Discret:R3, F.Cu at (141.0, 161.3)
- added R51: R, Discret:R3, F.Cu at (147.3, 157.5)
- added R52: R, Discret:R3, F.Cu at (163.8, 246.4)
- added R53: R, Discret:R3, F.Cu at (167.6, 240.0)
- added R54: R, Discret:R3, F.Cu at (171.4, 233.7)
- added R55: R, Discret:R3, F.Cu at (147.3, 281.9)
- added R56: R, Discret:R3, F.Cu at (153.7, 276.9)
- added U5: 74HC595, Sockets_DIP:DIP-16__300_ELL, F.Cu at (77.5, 188.0)
- added U6: 74HC595, Sockets_DIP:DIP-16__300_ELL, F.Cu at (148.6, 137.2)
- added U7: 74HC595, Sockets_DIP:DIP-16__300_ELL, F.Cu at (182.8, 168.0)
- moved R9 35.7 mm to (92.7, 281.9)
- moved R10 35.5 mm to (86.4, 276.9), turned to 180 degrees
- moved R13 18.3 mm to (82.5, 299.7), turned to 90 degrees
- moved R14 16.2 mm to (78.7, 297.2), turned to 90 degrees
- moved R15 14.9 mm to (74.9, 294.6), turned to 90 degrees
- moved R16 13.5 mm to (71.1, 290.8), turned to 90 degrees
- moved U2 8.68 mm to (69.8, 313.7), turned to 180 degrees
- moved R11 8.55 mm to (90.2, 304.8), turned to 90 degrees
- moved R12 4.48 mm to (86.4, 302.3), turned to 90 degrees
- moved D25 0.30 mm to (117.0, 216.1)
- moved D26 0.08 mm to (121.8, 216.1), turned to 180 degrees
Connections:
- U3 pad 9: Net-(U3-Pad9) -> LED_SERIAL_DATA_CHAIN4
- U4 pad 9: LED_SERIAL_DATA_CHAIN3 -> LED_SERIAL_DATA_CHAIN5
Routing:
- added copper zone on B.Cu, net GND
- added copper zone on F.Cu, net GND
Other:
- board outline added: 150 x 283.8 mm

Commit message: wip: tracing the minipinball PCB
Parts:
- moved R39 2.54 mm to (61.0, 167.6)
- moved R40 2.54 mm to (57.1, 167.6)
- turned R44 to 90 degrees
Routing:
- net LED_REGISTER_CLOCK: track 0.00 -> 267.4 mm, vias 0 -> 7
- net LED_SERIAL_CLOCK: track 0.00 -> 240.3 mm, vias 0 -> 3
- net LED_MASTER_RESET: track 0.00 -> 215.5 mm, vias 0 -> 3
- net VCC: track 0.00 -> 145.1 mm, vias 0 -> 4
- net Net-(D44-Pad1): track 0.00 -> 119.8 mm, vias 0 -> 3
- net LED_SERIAL_DATA_CHAIN6: track 0.00 -> 116.5 mm
- net Net-(D16-Pad1): track 0.00 -> 81.5 mm
- net Net-(D17-Pad1): track 0.00 -> 77.1 mm, vias 0 -> 1
- net Net-(D18-Pad1): track 0.00 -> 74.3 mm, vias 0 -> 1
- net Net-(R51-Pad1): track 0.00 -> 72.5 mm
- net Net-(D41-Pad1): track 0.00 -> 71.0 mm
- net Net-(R42-Pad1): track 0.00 -> 64.2 mm, vias 0 -> 2
- net Net-(D43-Pad1): track 0.00 -> 62.6 mm, vias 0 -> 2
- net Net-(R49-Pad1): track 0.00 -> 62.3 mm, vias 0 -> 1
- net Net-(R46-Pad1): track 0.00 -> 58.9 mm, vias 0 -> 2
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
Commit message: wip: tracing the minipinball PCB
Routing:
- net Net-(D15-Pad1): track 0.00 -> 108.3 mm, vias 0 -> 2
- net Net-(D6-Pad1): track 0.00 -> 93.6 mm, vias 0 -> 3
- net Net-(D14-Pad1): track 0.00 -> 76.1 mm, vias 0 -> 1
- net Net-(D5-Pad1): track 0.00 -> 67.6 mm, vias 0 -> 1
- net Net-(D29-Pad1): track 0.00 -> 66.8 mm
- net Net-(D4-Pad1): track 0.00 -> 62.0 mm, vias 0 -> 1
- net Net-(D7-Pad1): track 0.00 -> 57.8 mm
- net Net-(D1-Pad1): track 0.00 -> 57.2 mm
- net Net-(D3-Pad1): track 0.00 -> 53.8 mm, vias 0 -> 2
- net Net-(D11-Pad1): track 0.00 -> 53.7 mm
- net Net-(D2-Pad1): track 0.00 -> 49.8 mm, vias 0 -> 2
- net Net-(D32-Pad1): track 0.00 -> 27.2 mm
- net Net-(D31-Pad1): track 0.00 -> 16.3 mm
- net Net-(D30-Pad1): track 0.00 -> 16.3 mm
- net Net-(D52-Pad1): track 0.00 -> 15.8 mm
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