File: kicad/PARTYLand_miniplayfield.kicad_pcb (KiCad board)
At the start: 2 copper layers, 150 x 283.8 mm, 121 parts, among them P1 CONN_6, U1 74HC595, U2 74HC595, U3 74HC595, U4 74HC595, U5 74HC595, U6 74HC595, U7 74HC595

Commit message: work in progress...
Parts:
- removed G***: LOGO, partyland:playfield_inserts
- added R57: R, Discret:R3, F.Cu at (140.2, 318.3)
- added R58: R, Discret:R3, F.Cu at (136.7, 318.3)
- added R59: R, Discret:R3, F.Cu at (133.3, 318.3)
- added R60: R, Discret:R3, F.Cu at (129.8, 318.3)
- added R61: R, Discret:R3, F.Cu at (152.9, 332.7)
- added R62: R, Discret:R3, F.Cu at (156.5, 332.7)
- added R63: R, Discret:R3, F.Cu at (160.0, 332.7)
- added R64: R, Discret:R3, F.Cu at (163.6, 332.7)
- added SW1: SW_PUSH, Discret:SW_PUSH_SMALL, F.Cu at (121.7, 324.6)
- added SW2: SW_PUSH, Discret:SW_PUSH_SMALL, F.Cu at (58.9, 280.7)
- added SW3: SW_PUSH, Discret:SW_PUSH_SMALL, F.Cu at (67.6, 271.3)
- added SW4: SW_PUSH, Discret:SW_PUSH_SMALL, F.Cu at (173.0, 271.3)
- added SW5: SW_PUSH, Discret:SW_PUSH_SMALL, F.Cu at (182.1, 280.7)
- added SW6: SW_PUSH, Discret:SW_PUSH_SMALL, F.Cu at (87.4, 266.2)
- added SW7: SW_PUSH, Discret:SW_PUSH_SMALL, F.Cu at (153.4, 268.0)
- added SW8: SW_PUSH, Discret:SW_PUSH_SMALL, F.Cu at (194.1, 319.3)
- added U8: 74LS165, Sockets_DIP:DIP-16__300_ELL, F.Cu at (138.9, 333.0)
- P1: value CONN_6 -> CONN_10; footprint Pin_Headers:Pin_Header_Straight_1x06 -> Pin_Headers:Pin_Header_Angled_1x10
- moved P1 24.0 mm to (88.1, 325.9), turned to 270 degrees
Connections:
- P1 pad 2: LED_MASTER_RESET -> SWITCH_REGISTER_CLOCK
- P1 pad 3: LED_REGISTER_CLOCK -> SWITCH_SERIAL_DATA
- P1 pad 4: LED_SERIAL_DATA -> SWITCH_SERIAL_CLOCK
- P1 pad 5: LED_SERIAL_CLOCK -> GND
- P1 pad 6: VCC -> LED_MASTER_RESET
Routing:
- net Net-(D15-Pad1): track 108.3 -> 70.0 mm
- net Net-(D6-Pad1): track 93.6 -> 77.5 mm
